Commit message: add realsense camera for gazebo

File: husky_description/urdf/husky_macro.urdf.xacro (robot description, xacro)
@@ -5,7 +5,8 @@
   <xacro:arg name="laser_rpy" default="$(optenv CPR_LASER_RPY 0.0 0.0 0.0)" />
   <xacro:arg name="realsense_enabled" default="$(optenv CPR_REALSENSE 0)" />
+  <xacro:arg name="realsense_sgm_enabled" default="$(optenv CPR_REALSENSE_SGM 0)" />
   <xacro:arg name="realsense_xyz" default="$(optenv CPR_REALSENSE_XYZ 0 0 0)" />
   <xacro:arg name="realsense_rpy" default="$(optenv CPR_REALSENSE_RPY 0 0 0)" />
-  <xacro:arg name="realsense_mount" default="$(optenv CPR_REALSENSE_MOUNT_FRAME sensor_arch_mount_link)" />
+  <xacro:arg name="realsense_mount" default="$(optenv CPR_REALSENSE_MOUNT_FRAME top_plate_front_link)" />
   <xacro:property name="husky_front_bumper_extend" value="$(optenv HUSKY_FRONT_BUMPER_EXTEND 0)" />
   <xacro:property name="husky_rear_bumper_extend" value="$(optenv HUSKY_REAR_BUMPER_EXTEND 0)" />
@@ -17,5 +18,6 @@
   <xacro:include filename="$(find husky_description)/urdf/decorations.urdf.xacro" />
   <xacro:include filename="$(find husky_description)/urdf/wheel.urdf.xacro" />
-  <xacro:include filename="$(find husky_description)/urdf/accessories/intel_realsense.urdf.xacro"/>
+  <!-- <xacro:include filename="$(find husky_description)/urdf/accessories/intel_realsense.urdf.xacro"/> -->
+  <xacro:include filename="$(find husky_description)/urdf/accessories/d435.urdf.xacro"/>
   <!-- <xacro:include filename="$(find husky_description)/urdf/accessories/sick_lms1xx_mount.urdf.xacro"/> -->
   <xacro:include filename="$(find husky_description)/urdf/accessories/sensor_arch.urdf.xacro"/>
@@ -125,5 +127,7 @@
     </xacro:if> -->
     <!-- add the intel realsense to the topbar if needed -->
-    <xacro:if value="$(arg realsense_enabled)">
+    <xacro:property name="realsense_camera_enabled" value="$(arg realsense_enabled)" />
+    <xacro:property name="realsense_sgm_enabled" value="$(arg realsense_sgm_enabled)" />
+    <xacro:if value="${realsense_camera_enabled or realsense_sgm_enabled}">
       <link name="realsense_mountpoint"/>
       <joint name="realsense_mountpoint_joint" type="fixed">
@@ -132,5 +136,5 @@
         <child link="realsense_mountpoint" />
       </joint>
-      <xacro:intel_realsense_mount prefix="camera" topic="realsense" parent_link="realsense_mountpoint"/>
+      <xacro:intel_realsense_mount prefix="camera" parent_link="realsense_mountpoint"/>
     </xacro:if>
     <ros2_control name="${prefix}husky_hardware" type="system">
