Commit message: add wheel slip

File: husky_description/urdf/husky.urdf.xacro (robot description, xacro)
@@ -40,4 +40,44 @@
       </sensor>
     </gazebo>
+    <gazebo>
+      <plugin name="gazebo_ros_p3d" filename="libgazebo_ros_p3d.so">
+        <ros>
+          <namespace>$(arg prefix)</namespace>
+          <remapping>odom:=ground_truth</remapping>
+        </ros>
+        <body_name>base_link</body_name>
+        <update_rate>10</update_rate>
+      </plugin>
+    </gazebo>
+    <xacro:if value="$(arg husky_wheel_slip)">
+      <gazebo>
+        <plugin filename="libgazebo_ros_wheel_slip.so" name="wheels_slip">
+          <wheel link_name="front_left_wheel">
+            <slip_compliance_lateral>1.0</slip_compliance_lateral>
+            <slip_compliance_longitudinal>1.0</slip_compliance_longitudinal>
+            <wheel_normal_force>113</wheel_normal_force>
+            <wheel_radius>0.1651</wheel_radius>
+          </wheel>
+          <wheel link_name="front_right_wheel">
+            <slip_compliance_lateral>1.0</slip_compliance_lateral>
+            <slip_compliance_longitudinal>1.0</slip_compliance_longitudinal>
+            <wheel_normal_force>113</wheel_normal_force>
+            <wheel_radius>0.1651</wheel_radius>
+          </wheel>
+          <wheel link_name="rear_left_wheel">
+            <slip_compliance_lateral>1.0</slip_compliance_lateral>
+            <slip_compliance_longitudinal>1.0</slip_compliance_longitudinal>
+            <wheel_normal_force>113</wheel_normal_force>
+            <wheel_radius>0.1651</wheel_radius>
+          </wheel>
+          <wheel link_name="rear_right_wheel">
+            <slip_compliance_lateral>1.0</slip_compliance_lateral>
+            <slip_compliance_longitudinal>1.0</slip_compliance_longitudinal>
+            <wheel_normal_force>113</wheel_normal_force>
+            <wheel_radius>0.1651</wheel_radius>
+          </wheel>
+        </plugin>
+      </gazebo>
+    </xacro:if>
   </xacro:if>
   <!-- Optional custom includes. -->

File: husky_description/urdf/husky_macro.urdf.xacro (robot description, xacro)
@@ -9,4 +9,5 @@
   <xacro:arg name="realsense_rpy" default="$(optenv CPR_REALSENSE_RPY 0 0 0)" />
   <xacro:arg name="realsense_mount" default="$(optenv CPR_REALSENSE_MOUNT_FRAME top_plate_front_link)" />
+  <xacro:arg name="husky_wheel_slip" default="$(optenv HUSKY_WHEEL_SLIP 0)" />
   <xacro:property name="husky_front_bumper_extend" value="$(optenv HUSKY_FRONT_BUMPER_EXTEND 0)" />
   <xacro:property name="husky_rear_bumper_extend" value="$(optenv HUSKY_REAR_BUMPER_EXTEND 0)" />
@@ -30,5 +31,5 @@
     <!-- Wheel Mounting Positions -->
     <xacro:property name="wheelbase" value="0.5120" />
-    <xacro:property name="track" value="0.5708" />
+    <xacro:property name="track" value="0.555" />
     <xacro:property name="wheel_vertical_offset" value="0.03282" />
     <!-- Wheel Properties -->

File: husky_description/urdf/wheel.urdf.xacro (robot description, xacro)
@@ -21,11 +21,13 @@
       </collision>
     </link>
-    <gazebo reference="${wheel_prefix}_wheel">
-      <mu1 value="1.0"/>
-      <mu2 value="0.5"/>
-      <kp value="10000000.0" />
-      <kd value="1.0" />
-      <fdir1 value="1 0 0"/>
-    </gazebo>
+    <xacro:unless value="$(arg husky_wheel_slip)">
+      <gazebo reference="${wheel_prefix}_wheel">
+        <mu1 value="1.0"/>
+        <mu2 value="0.5"/>
+        <kp value="10000000.0" />
+        <kd value="1.0" />
+        <fdir1 value="1 0 0"/>
+      </gazebo>
+    </xacro:unless>
     <joint name="${wheel_prefix}_wheel_joint" type="continuous">
       <parent link="base_link"/>

Commit message: add collision link and collision detection plugin

File: husky_description/urdf/husky.urdf.xacro (robot description, xacro)
@@ -50,4 +50,20 @@
       </plugin>
     </gazebo>
+    <gazebo reference="collision_link">
+      <sensor name='collision_sensor' type='contact'>
+        <update_rate>10</update_rate>
+        <contact>
+          <!-- <collision>base_link_collision</collision> -->
+          <collision>base_link_fixed_joint_lump__collision_link_collision_2</collision>
+        </contact>
+        <plugin name="collision_sensor" filename="libgazebo_ros_collision.so">
+          <ros>
+            <namespace>husky</namespace>
+          </ros>
+          <frame_name>collision_link</frame_name>
+          <terrain_name>terrain2</terrain_name>
+        </plugin>
+      </sensor>
+    </gazebo>
     <xacro:if value="$(arg husky_wheel_slip)">
       <gazebo>

File: husky_description/urdf/husky_macro.urdf.xacro (robot description, xacro)
@@ -72,4 +72,17 @@
       </inertial>
     </link>
+    <link name="${prefix}collision_link">
+      <collision>
+        <origin xyz="0 0 0" rpy="0 0 0" />
+        <geometry>
+          <box size="${base_x_size+ 0.04} ${track + wheel_length + 0.04} ${base_z_size/2}"/>
+        </geometry>
+      </collision>
+    </link>
+    <joint name="${prefix}collision_joint" type="fixed">
+      <origin xyz="0 0 0" rpy="0 0 0" />
+      <parent link="${prefix}base_link" />
+      <child link="${prefix}collision_link" />
+    </joint>
     <joint name="${prefix}inertial_joint" type="fixed">
       <origin xyz="0 0 0" rpy="0 0 0" />

File: husky_description/urdf/wheel.urdf.xacro (robot description, xacro)
@@ -14,5 +14,5 @@
         </geometry>
       </visual>
-      <collision>
+      <collision name="${wheel_prefix}_wheel_c">
         <origin xyz="0 0 0" rpy="${M_PI/2} 0 0" />
         <geometry>
